File: Basic-150-MHz-Telemetry-Transmitter-SMD/Basic-150-MHz-Telemetry-Transmitter-SMD.kicad_sch (KiCad schematic)
At the start: 11 parts

Commit message: smd ver
Parts:
- removed Q1: (no value), symbol Transistor_BJT:2N3904
- added C3: C_Small, Capacitor_SMD:C_0805_2012Metric_Pad1.18x1.45mm_HandSolder, symbol Device:C_Small
- added Q1: (no value), symbol Transistor_BJT:MMBT3904
- C1, C2, CP1: footprint Capacitor_THT:C_Disc_D10.0mm_W2.5mm_P5.00mm -> (none)
- J1: value (none) -> input/output; footprint (none) -> Connector_PinHeader_2.54mm:PinHeader_1x03_P2.54mm_Vertical
- J2: value (none) -> Antenna
- L1: value (none) -> INDUCTOR
Connections:
- net GND: now also Q1.2 (E)
- net at R1.2, Y1.2: now also Q1.1 (B)
- net at C2.1, L2.2, Y1.1: now also C3.1, Q1.3 (C); no longer J2.2 (Pin_2)
- new net: C3.2, J2.2 (Pin_2)

Commit message: f
Parts:
- C1: value C_Small -> (none); footprint (none) -> Capacitor_SMD:C_0805_2012Metric_Pad1.18x1.45mm_HandSolder
- C2, C3: value C_Small -> (none)
- CP1, RP1: footprint (none) -> Capacitor_SMD:C_0805_2012Metric_Pad1.18x1.45mm_HandSolder
- L1, L2: value INDUCTOR -> (none); footprint (none) -> Inductor_SMD:L_0805_2012Metric_Pad1.15x1.40mm_HandSolder
- Q1: value (none) -> MMBT3904; footprint (none) -> Package_TO_SOT_SMD:SOT-23
- R1: value R_Small -> (none); footprint (none) -> Capacitor_SMD:C_0805_2012Metric_Pad1.18x1.45mm_HandSolder
- Y1: value (none) -> Crystal_GND3; footprint (none) -> Crystal:Crystal_SMD_SeikoEpson_FA238V-4Pin_3.2x2.5mm_HandSoldering
Other:
- note added: "Mouser filters: Crystal: https://ro.mouser.com/c/passive-components/frequency-control-timing-devices/crystals/?frequency=50%20MHz&package%20%2F%20case=3.2%20mm%20x%202.5%20mm~~3.2%20mm%20x%202.5%20mm%20x%200.7%20mm&termination%20style=SMD%2FSMT&instock=y&active=y&sort=pricing&rp=passive-components%2Ffrequency-control-timing-devices%2Fcrystals%7C~Package%20%2F%20Case L2 https://ro.mouser.com/c/pas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"
Changed lines of the file:
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@@
+    (effects (font (size 1.27 1.27)) (justify left bottom))
+  )
+  (text "Mouser filters:\n\nCrystal:   https://ro.mouser.com/c/passive-components/frequency-control-timing-devices/crystals/?frequency=50%20MHz&package%20%2F%20case=3.2%20mm%20x%202.5%20mm~~3.2%20mm%20x%202.5%20mm%20x%200.7%20mm&termination%20style=SMD%2FSMT&instock=y&active=y&sort=pricing&rp=passive-components%2Ffrequency-control-timing-devices%2Fcrystals%7C~Package%20%2F%20Case\nL2  https://ro.mouser.com/c/passive-components/inductors-chokes-coils/fixed-inductors/?inductance=1%20uH&package%20%2F%20case=0805%20%282012%20metric%29~~0806%20%282016%20metric%29&product=RF%20Inductors&termination%20style=SMD%2FSMT&instock=y&sort=pricing&rp=passive-components%2Finductors-chokes-coils%2Ffixed-inductors%7C~Package%20%2F%20Case\nL1  https://ro.mouser.com/c/passive-components/inductors-chokes-coils/fixed-inductors/?inductance=100%20nH&package%20%2F%20case=0805%20%282012%20metric%29~~0805%20%282015%20metric%29&product=RF%20Inductors&termination%20style=SMD%2FSMT&instock=y&sort=pricing&rp=passive-components%2Finductors-chokes-coils%2Ffixed-inductors%7C~Package%20%2F%20Case\n"
+    (at 24.13 142.875 0)
     (effects (font (size 1.27 1.27)) (justify left bottom))
   )
@@
       (effects (font (size 1.27 1.27)) (justify right))
     )
-    (property "Value" "C_Small" (id 1) (at 74.93 74.295 0)
-      (effects (font (size 1.27 1.27)) (justify right))
-    )
-    (property "Footprint" "" (id 2) (at 71.755 72.39 0)
+    (property "Value" "" (id 1) (at 74.93 74.295 0)
+      (effects (font (size 1.27 1.27)) (justify right))
+    )
+    (property "Footprint" "Capacitor_SMD:C_0805_2012Metric_Pad1.18x1.45mm_HandSolder" (id 2) (at 71.755 72.39 0)
       (effects (font (size 1.27 1.27)) hide)
     )
@@
       (effects (font (size 1.27 1.27)) (justify left))
     )
-    (property "Value" "" (id 1) (at 98.425 90.17 90)
-      (effects (font (size 1.27 1.27)) (justify left))
-    )
-    (property "Footprint" "" (id 2) (at 106.045 95.885 0)
+    (property "Value" "Crystal_GND3" (id 1) (at 98.425 90.17 90)
+      (effects (font (size 1.27 1.27)) (justify left))
+    )
+    (property "Footprint" "Crystal:Crystal_SMD_SeikoEpson_FA238V-4Pin_3.2x2.5mm_HandSoldering" (id 2) (at 106.045 95.885 0)
       (effects (font (size 1.27 1.27)) hide)
     )
@@
     (in_bom yes) (on_board yes) (fields_autoplaced)
     (property "Reference" "L1" (id 0) (at 104.775 55.88 0))
-    (property "Value" "INDUCTOR" (id 1) (at 104.775 58.42 0))
-    (property "Footprint" "" (id 2) (at 104.775 62.865 0)
+    (property "Value" "" (id 1) (at 104.775 58.42 0))
+    (property "Footprint" "Inductor_SMD:L_0805_2012Metric_Pad1.15x1.40mm_HandSolder" (id 2) (at 104.775 62.865 0)
       (effects (font (size 1.27 1.27)) hide)
     )
@@
       (effects (font (size 1.27 1.27)) (justify left))
     )
-    (property "Footprint" "" (id 2) (at 88.265 82.55 0)
+    (property "Footprint" "Capacitor_SMD:C_0805_2012Metric_Pad1.18x1.45mm_HandSolder" (id 2) (at 88.265 82.55 0)
       (effects (font (size 1.27 1.27)) hide)
     )
@@
       (effects (font (size 1.27 1.27)) (justify right))
     )
-    (property "Value" "C_Small" (id 1) (at 104.14 73.66 0)
+    (property "Value" "" (id 1) (at 104.14 73.66 0)
       (effects (font (size 1.27 1.27)) (justify right))
     )
@@
       (effects (font (size 1.27 1.27)) (justify left))
     )
-    (property "Footprint" "" (id 2) (at 88.265 73.025 0)
+    (property "Footprint" "Capacitor_SMD:C_0805_2012Metric_Pad1.18x1.45mm_HandSolder" (id 2) (at 88.265 73.025 0)
       (effects (font (size 1.27 1.27)) hide)
     )
@@
     (in_bom yes) (on_board yes)
     (property "Reference" "R1" (id 0) (at 99.06 109.855 90))
-    (property "Value" "R_Small" (id 1) (at 99.06 112.395 90))
-    (property "Footprint" "" (id 2) (at 99.695 106.045 0)
+    (property "Value" "" (id 1) (at 99.06 112.395 90))
+    (property "Footprint" "Capacitor_SMD:C_0805_2012Metric_Pad1.18x1.45mm_HandSolder" (id 2) (at 99.695 106.045 0)
       (effects (font (size 1.27 1.27)) hide)
     )
@@
       (effects (font (size 1.27 1.27)) (justify left))
     )
-    (property "Value" "INDUCTOR" (id 1) (at 123.19 73.6599 90)
-      (effects (font (size 1.27 1.27)) (justify left))
-    )
-    (property "Footprint" "" (id 2) (at 121.285 72.39 0)
+    (property "Value" "" (id 1) (at 123.19 73.6599 90)
+      (effects (font (size 1.27 1.27)) (justify left))
+    )
+    (property "Footprint" "Inductor_SMD:L_0805_2012Metric_Pad1.15x1.40mm_HandSolder" (id 2) (at 121.285 72.39 0)
       (effects (font (size 1.27 1.27)) hide)
     )
@@
       (effects (font (size 1.27 1.27)) (justify left))
     )
-    (property "Value" "" (id 1) (at 121.285 107.3149 0)
-      (effects (font (size 1.27 1.27)) (justify left))
-    )
-    (property "Footprint" "" (id 2) (at 121.285 107.95 0)
+    (property "Value" "MMBT3904" (id 1) (at 121.285 107.3149 0)
+      (effects (font (size 1.27 1.27)) (justify left))
+    )
+    (property "Footprint" "Package_TO_SOT_SMD:SOT-23" (id 2) (at 121.285 107.95 0)
       (effects (font (size 1.27 1.27) italic) (justify left) hide)
     )
@@
       (effects (font (size 1.27 1.27)) (justify right))
     )
-    (property "Value" "C_Small" (id 1) (at 127 89.535 90)
+    (property "Value" "" (id 1) (at 127 89.535 90)
       (effects (font (size 1.27 1.27)) (justify right))
     )
@@
     )
     (path "/0c544a8c-9f45-4205-9bca-1d91c95d58ef"
-      (reference "C1") (unit 1) (value "C_Small") (footprint "Capacitor_SMD:C_0805_2012Metric_Pad1.18x1.45mm_HandSolder")
+      (reference "C1") (unit 1) (value "100n") (footprint "Capacitor_SMD:C_0805_2012Metric_Pad1.18x1.45mm_HandSolder")
     )
     (path "/96ef76a5-90c3-4767-98ba-2b61887e28d3"
-      (reference "C2") (unit 1) (value "C_Small") (footprint "Capacitor_SMD:C_0805_2012Metric_Pad1.18x1.45mm_HandSolder")
+      (reference "C2") (unit 1) (value "15p") (footprint "Capacitor_SMD:C_0805_2012Metric_Pad1.18x1.45mm_HandSolder")
     )
     (path "/ed26d778-1613-45ec-a8f9-f4108a089f4f"
-      (reference "C3") (unit 1) (value "C_Small") (footprint "Capacitor_SMD:C_0805_2012Metric_Pad1.18x1.45mm_HandSolder")
+      (reference "C3") (unit 1) (value "2p2") (footprint "Capacitor_SMD:C_0805_2012Metric_Pad1.18x1.45mm_HandSolder")
     )
     (path "/765684c2-53b3-4ef7-bd1b-7a4a73d87b76"
@@
     )
     (path "/662bafcb-dcfb-4471-a8a9-f5c777fdf249"
-      (reference "L1") (unit 1) (value "INDUCTOR") (footprint "Inductor_SMD:L_0805_2012Metric_Pad1.15x1.40mm_HandSolder")
+      (reference "L1") (unit 1) (value "100n") (footprint "Inductor_SMD:L_0805_2012Metric_Pad1.15x1.40mm_HandSolder")
     )
     (path "/bb8162f0-99c8-4884-be5b-c0d0c7e81ff6"
-      (reference "L2") (unit 1) (value "INDUCTOR") (footprint "Inductor_SMD:L_0805_2012Metric_Pad1.15x1.40mm_HandSolder")
+      (reference "L2") (unit 1) (value "1u") (footprint "Inductor_SMD:L_0805_2012Metric_Pad1.15x1.40mm_HandSolder")
     )
     (path "/cdd691ae-ae40-4f3b-84d4-cc54b1b75971"
@@
     )
     (path "/9c2999b2-1cf1-4204-9d23-243401b77aa3"
-      (reference "R1") (unit 1) (value "R_Small") (footprint "Capacitor_SMD:C_0805_2012Metric_Pad1.18x1.45mm_HandSolder")
+      (reference "R1") (unit 1) (value "390k") (footprint "Capacitor_SMD:C_0805_2012Metric_Pad1.18x1.45mm_HandSolder")
     )
     (path "/981ff4de-0330-4757-b746-0cb983df5e7c"
