File: Basic-150-MHz-Telemetry-Transmitter-SMD/Basic-150-MHz-Telemetry-Transmitter-SMD.kicad_pcb (KiCad board)
At the start: 2 copper layers, 22 x 15 mm, 12 parts, among them J1 input/output, J2 Antenna, Q1 MMBT3904, Y1 Crystal_GND3

Commit message: y
Parts:
- added ?: , Aesthetics:OSHW-LOGO-M, F.Cu at (58.5, 51.1)
- added G***: LOGO, LOGO, B.Cu at (58.4, 51.1)

Commit message: fixes
Parts:
- added kibuzzard-632D4E48: G***, kibuzzard-632D4E48, B.Cu at (42.9, 50.3)
- added kibuzzard-632D4E55: G***, kibuzzard-632D4E55, B.Cu at (44.9, 45.9)
- added kibuzzard-632D4E64: G***, kibuzzard-632D4E64, B.Cu at (45.0, 42.1)
-  : renamed from G***
