File: Basic-150-MHz-Telemetry-Transmitter-THT/Basic-150-MHz-Telemetry-Transmitter-THT.kicad_pcb (KiCad board)
At the start: 2 copper layers, 33.8 x 21.8 mm, 11 parts, among them J1 input/output, J2 Antenna, Q1 2N3904, Y1 Crystal_GND3

Commit message: y
Parts:
- added ?: , Aesthetics:OSHW-LOGO-M, F.Cu at (82.4, 112.2)
- added G***: LOGO, LOGO, B.Cu at (82.5, 112.4)

Commit message: fixes
Parts:
- added kibuzzard-632D4D9D: G***, kibuzzard-632D4D9D, B.Cu at (56.7, 102.5)
- added kibuzzard-632D4DBD: G***, kibuzzard-632D4DBD, B.Cu at (56.7, 98.3)
- added kibuzzard-632D4DD2: G***, kibuzzard-632D4DD2, B.Cu at (55.0, 107.1)
